File: KiCAD_files/V_Neutral.kicad_sch (KiCad schematic)
At the start: 0 parts

Commit message: save before starting routing
Other:
- title: (none) -> Inverter V0.1
Changed lines of the file:
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@@
 (kicad_sch (version 20230121) (generator eeschema)
   (paper "A4")
+  (title_block
+    (title "Inverter V0.1")
+    (comment 1 "TWR")
+  )
 )
