File: KiCAD_files/inverter.kicad_pcb (KiCad board)
At the start: 6 copper layers, 100 x 220.5 mm, 406 parts, among them J101 Wago 4 contacts, J103 2604-1102, J104 2604-1102, J105 2604-1102, J106 2604-1102, J107 2604-1102, J108 2604-1102, J403 RJ45_LED_Shielded, J404 RJ45_LED_Shielded, J405 Conn_01x02_Male, J406 Conn_01x02_Male, J501 Conn_01x03, J901 Conn_01x05, Q501 60V N channel, Q502 TK13P25D,RQ, Q601 IPD200N15N3, Q602 IPD200N15N3, Q701 IPD200N15N3, Q702 IPD200N15N3, Q801 IPD200N15N3, Q802 IPD200N15N3, T501 PA2467NL, U201 AMC1311DWV, U202 +-20A Hall, U203 OPA316, U204 OPA316, U301 AP1117-50, U302 MCP1799T-5002H/TT, U401 OwnTech_SPIN, U402 TCAN334GDR, U405 LTC2850xS8, U406 OPA2277, U407 OPA316, U410 TS5A3357DCUT, U490 OPA316, U501 NCP12700, U502 FODM217A, U503 TL431MFDT,215, U601 AMC1100DUB, U602 FODM217A, U603 UCC21222DR, U604 OPA316, U605 ACS730KLCTR-20AB, U606 OPA316, U701 AMC1100DUB, U702 FODM217A, U703 UCC21222DR, U704 OPA316, U705 ACS730KLCTR-20AB, U706 OPA316, U801 AMC1100DUB, U802 FODM217A, U803 UCC21222DR, U804 OPA316, U805 ACS730KLCTR-20AB, U806 OPA316, U901 ISO6740DW

Commit message: dev
Parts:
- moved R716 172.6 mm to (60.3, 144.0), turned to -90 degrees
- moved R717 168.8 mm to (60.3, 147.5), turned to -90 degrees
- moved C701 167.0 mm to (62.5, 147.4), turned to -90 degrees
- moved U701 160.4 mm to (69.8, 147.5), turned to 0 degrees
- moved R713 155.8 mm to (80.2, 144.3), turned to 0 degrees
- moved C706 154.4 mm to (77.1, 147.5), turned to -90 degrees
- moved R711 153.3 mm to (80.2, 146.4), turned to 0 degrees
- moved R712 150.5 mm to (80.2, 148.7), turned to 0 degrees
- moved C710 149.5 mm to (76.9, 151.8), turned to -90 degrees
- moved R715 147.9 mm to (78.9, 151.8), turned to -90 degrees
- moved U704 146.0 mm to (81.3, 151.8), turned to -90 degrees
- moved U410 139.5 mm to (101.6, 174.2)
- moved C420 139.4 mm to (101.6, 171.8)
- moved C721 136.8 mm to (51.0, 102.0), turned to 180 degrees
- moved R425 133.7 mm to (102.3, 176.4), turned to 180 degrees
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Routing:
- net /Phase1/SW_Node: track 16.2 -> 214.0 mm
- net /HRTIM_CHA2: track 293.2 -> 109.4 mm
- net /V_{IHigh_sense}: track 102.7 -> 175.6 mm, vias 1 -> 2
- net Net-(F601-Pad1): track 72.9 -> 0.00 mm, vias 9 -> 0
- net DGND: track 196.1 -> 168.3 mm, vias 73 -> 66
- net +5V_DGND: track 241.5 -> 219.9 mm, vias 48 -> 32
- net /HRTIM_CHA1: track 125.8 -> 106.4 mm
- net +5V_PGND: track 46.6 -> 36.0 mm
- net /I_{I3Low_sense}: track 18.4 -> 7.85 mm
- net Net-(U806-+): track 7.92 -> 0.00 mm
- net Net-(U606--): track 6.29 -> 0.00 mm
- net Net-(U603-INB): track 5.62 -> 0.00 mm
- net Net-(U603-INA): track 5.40 -> 0.00 mm
- net Net-(U806--): track 12.6 -> 7.85 mm
- net Net-(D801-A): track 16.3 -> 20.9 mm
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- removed copper zone on F.Cu, net Net-(F601-Pad1)
- removed copper zone on F.Cu, net Net-(F701-Pad1)
- removed copper zone on F.Cu, net Net-(F801-Pad1)
- removed copper zone on F.Cu, net Net-(L701-Pad1)
Other:
- board size 100 x 220.5 mm -> 100 x 220 mm

Commit message: dev
Parts:
- removed C620, C621, C720, C721, C820, C821: 33uF, Capacitor_SMD:CP_Elec_10x10.5
- removed H102, H109: M2.5, MountingHole:MountingHole_2.7mm_M2.5_DIN965_Pad_TopOnly
- removed J105, J107: 2604-1102, Footprints:WAGO-2604-1102
- added C205: 33uF, Capacitor_SMD:CP_Elec_10x10.5, F.Cu at (52.0, 157.1)
- added C206: 33uF, Capacitor_SMD:CP_Elec_10x10.5, F.Cu at (52.0, 144.8)
- added C208: 33uF, Capacitor_SMD:CP_Elec_10x10.5, F.Cu at (52.0, 132.6)
- added C210: 33uF, Capacitor_SMD:CP_Elec_10x10.5, F.Cu at (52.0, 120.4)
- added C211: 33uF, Capacitor_SMD:CP_Elec_10x10.5, F.Cu at (52.0, 108.2)
- added C212: 33uF, Capacitor_SMD:CP_Elec_10x10.5, F.Cu at (52.0, 96.0)
- added H104: M2.5, MountingHole:MountingHole_2.7mm_M2.5_DIN965_Pad_TopOnly, F.Cu at (91.0, 125.2)
- added H104: M2.5, MountingHole:MountingHole_2.7mm_M2.5_DIN965_Pad_TopOnly, F.Cu at (63.4, 100.4)
- added H104: M2.5, MountingHole:MountingHole_2.7mm_M2.5_DIN965_Pad_TopOnly, F.Cu at (136.4, 156.0)
- added H104: M2.5, MountingHole:MountingHole_2.7mm_M2.5_DIN965_Pad_TopOnly, F.Cu at (91.0, 156.0)
- added H104: M2.5, MountingHole:MountingHole_2.7mm_M2.5_DIN965_Pad_TopOnly, F.Cu at (119.2, 125.0)
- C202, C203, C601, C606, C611, C701, C706, C711, C801, C806, C811: footprint Capacitor_SMD:C_1206_3216Metric -> Capacitor_SMD:C_0603_1608Metric
- J103: value 2604-1102 -> Wago 6 contacts; footprint Footprints:WAGO-2604-1102 -> Footprints:WAGO-2604-1106
- J901: footprint Connector_JST:JST_EH_B6B-EH-A_1x06_P2.50mm_Vertical -> Connector_JST:JST_EH_B5B-EH-A_1x05_P2.50mm_Vertical
- U901: value ISO6740DW -> Si8640BB-B-IS1; footprint Footprints:SOIC-16W_7.5x12.8mm_P1.27mm -> Package_SO:SOIC-16_3.9x9.9mm_P1.27mm
- moved N101 249.8 mm to (-233.0, -84.5)
- moved H104 111.9 mm to (63.2, 125.2)
- moved J103 86.5 mm to (89.8, 169.2)
- moved R816 68.8 mm to (117.7, 144.3), turned to 0 degrees
- moved R817 64.3 mm to (118.4, 146.6), turned to -90 degrees
- moved C801 63.5 mm to (120.7, 141.1)
- moved R450 61.5 mm to (107.2, 65.8)
- moved U801 59.2 mm to (125.5, 146.7), turned to 0 degrees
- moved TH403 58.7 mm to (106.5, 67.6), turned to -90 degrees
- moved R813 58.3 mm to (135.6, 143.7)
- moved R811 57.6 mm to (133.2, 145.5), turned to 0 degrees
- moved C806 56.6 mm to (133.0, 142.9), turned to 0 degrees
- moved R812 54.5 mm to (133.2, 147.9), turned to 0 degrees
- moved R815 50.4 mm to (133.2, 149.5), turned to 0 degrees
- moved U804 50.1 mm to (136.6, 146.7), turned to 0 degrees
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Connections:
- C202 pad 1: +5V_DGND -> DGND
- C202 pad 2: DGND -> +5V_DGND
- C203 pad 1: +5V_DGND -> DGND
- C203 pad 2: DGND -> +5V_DGND
- C601 pad 1: +5V_PGND -> PGND
- C601 pad 2: PGND -> +5V_PGND
- C701 pad 1: +5V_PGND -> PGND
- C701 pad 2: PGND -> +5V_PGND
- C801 pad 1: +5V_PGND -> PGND
- C801 pad 2: PGND -> +5V_PGND
- U901 pad 12: /HALL3 -> /HALL1
- U901 pad 14: /HALL1 -> /HALL3
- U901 pad 3: /Hall_Sensor/HALL1_PGND -> /Hall_Sensor/HALL3_PGND
- U901 pad 5: /Hall_Sensor/HALL3_PGND -> /Hall_Sensor/HALL1_PGND
Routing:
- net /HRTIM_CHE2: track 0.00 -> 172.3 mm
- net +5V_DGND: track 219.9 -> 56.0 mm, vias 32 -> 20
- net /HRTIM_CHE1: track 0.00 -> 141.8 mm
- net PGND: track 175.6 -> 58.2 mm, vias 87 -> 238
- net /VRef: track 106.0 -> 2.24 mm, vias 2 -> 1
- net /~{STBY1}: track 0.67 -> 104.0 mm, vias 1 -> 7
- net /MCU/Temp3: track 0.00 -> 98.0 mm, vias 0 -> 2
- net /V_{IHigh_sense}: track 175.6 -> 82.1 mm, vias 2 -> 1
- net DGND: track 168.3 -> 75.1 mm, vias 66 -> 88
- net /HRTIM_CHA1: track 106.4 -> 185.1 mm
- net /HRTIM_CHA2: track 109.4 -> 185.1 mm
- net /V_{I1Low_sense}: track 122.8 -> 182.6 mm, vias 1 -> 3
- net +12V_PGND: track 59.2 -> 0.00 mm, vias 27 -> 32
- net Net-(F701-Pad1): track 145.8 -> 91.4 mm, vias 2 -> 34
- net /I_{I1Low_sense}: track 72.5 -> 115.4 mm, vias 1 -> 2
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- added copper zone on F.Cu, net /Feeder/VIN
- added copper zone on In3.Cu, net /Feeder/VIN
- added copper zone on F.Cu, net /High_side/V_{IHighIN}
- added copper zone on In3.Cu, net /High_side/V_{IHighIN}
- added copper zone on F.Cu, net /Phase A
- added copper zone on In3.Cu, net /Phase A
- added copper zone on F.Cu, net /Phase B
- added copper zone on In3.Cu, net /Phase B
- added copper zone on F.Cu, net /Phase C
- added copper zone on In3.Cu, net /Phase C
- added copper zone on F.Cu, net Net-(F201-Pad2)
- added copper zone on In3.Cu, net Net-(F201-Pad2)
- added copper zone on F.Cu, net Net-(F601-Pad1)
- added copper zone on In3.Cu, net Net-(F601-Pad1)
- added copper zone on F.Cu, net Net-(F701-Pad1)
- added copper zone on In3.Cu, net Net-(F701-Pad1)
- added copper zone on F.Cu, net Net-(F801-Pad1)
- added copper zone on In3.Cu, net Net-(F801-Pad1)
- added copper zone on F.Cu, net Net-(L601-Pad1)
- added copper zone on F.Cu, net Net-(L701-Pad1)
- added copper zone on F.Cu, net Net-(L801-Pad1)
- removed copper zone on In2.Cu, net +3.3V_DGND
- removed copper zone on F.Cu, net +5V_DGND
- removed copper zone on B.Cu, net PGND
- removed copper zone on In1.Cu, net PGND
- removed copper zone on In4.Cu, net PGND
Other:
- board size 100 x 220 mm -> 100 x 160 mm

Commit message: dev
Parts:
- added C620: 33uF, Capacitor_SMD:CP_Elec_10x10.5, F.Cu at (-8.27, 102.3)
- added C621: 33uF, Capacitor_SMD:CP_Elec_10x10.5, F.Cu at (-8.27, 114.4)
- added C720: 33uF, Capacitor_SMD:CP_Elec_10x10.5, F.Cu at (-35.0, 102.3)
- added C721: 33uF, Capacitor_SMD:CP_Elec_10x10.5, F.Cu at (-35.0, 114.4)
- added C820: 33uF, Capacitor_SMD:CP_Elec_10x10.5, F.Cu at (-35.0, 128.4)
- added C821: 33uF, Capacitor_SMD:CP_Elec_10x10.5, F.Cu at (-35.0, 140.5)
- added H102: M2.5, MountingHole:MountingHole_2.7mm_M2.5_DIN965_Pad_TopOnly, F.Cu at (-7.00, 141.8)
- added H104: M2.5, MountingHole:MountingHole_2.7mm_M2.5_DIN965_Pad_TopOnly, F.Cu at (119.2, 100.4)
- added H104: M2.5, MountingHole:MountingHole_2.7mm_M2.5_DIN965_Pad_TopOnly, F.Cu at (91.0, 100.4)
- added H109: M2.5, MountingHole:MountingHole_2.7mm_M2.5_DIN965_Pad_TopOnly, F.Cu at (-7.00, 148.0)
- added TP201: TestPoint, Footprints:TestPoint_THTPad_D1.5mm_Drill0.7mm, F.Cu at (4.30, 124.2)
- added TP202: TestPoint, Footprints:TestPoint_THTPad_D1.5mm_Drill0.7mm, F.Cu at (4.30, 127.8)
- added TP203: TestPoint, Footprints:TestPoint_THTPad_D1.5mm_Drill0.7mm, F.Cu at (4.30, 131.3)
- added TP204: TestPoint, Footprints:TestPoint_THTPad_D1.5mm_Drill0.7mm, F.Cu at (4.30, 134.8)
- added TP418: TestPoint, Footprints:TestPoint_THTPad_D1.5mm_Drill0.7mm, F.Cu at (-8.35, 131.3)
- added TP419: TestPoint, Footprints:TestPoint_THTPad_D1.5mm_Drill0.7mm, F.Cu at (-8.35, 134.8)
- added TP450: TestPoint, Footprints:TestPoint_THTPad_D1.5mm_Drill0.7mm, F.Cu at (-4.80, 124.2)
- added TP451: TestPoint, Footprints:TestPoint_THTPad_D1.5mm_Drill0.7mm, F.Cu at (-4.80, 127.8)
- added TP452: TestPoint, Footprints:TestPoint_THTPad_D1.5mm_Drill0.7mm, F.Cu at (-4.80, 131.3)
- added TP453: TestPoint, Footprints:TestPoint_THTPad_D1.5mm_Drill0.7mm, F.Cu at (-4.80, 134.8)
- added TP491: TestPoint, Footprints:TestPoint_THTPad_D1.5mm_Drill0.7mm, F.Cu at (-1.25, 124.2)
- added TP492: TestPoint, Footprints:TestPoint_THTPad_D1.5mm_Drill0.7mm, F.Cu at (-1.25, 127.8)
- added TP493: TestPoint, Footprints:TestPoint_THTPad_D1.5mm_Drill0.7mm, F.Cu at (-1.25, 131.3)
- added TP601: TestPoint, Footprints:TestPoint_THTPad_D1.5mm_Drill0.7mm, F.Cu at (0.68, 98.1)
- added TP602: TestPoint, Footprints:TestPoint_THTPad_D1.5mm_Drill0.7mm, F.Cu at (0.68, 101.7)
- added TP603: TestPoint, Footprints:TestPoint_THTPad_D1.5mm_Drill0.7mm, F.Cu at (0.68, 105.2)
- added TP604: TestPoint, TestPoint:TestPoint_Pad_D1.0mm, F.Cu at (7.53, 97.8)
- added TP605: TestPoint, TestPoint:TestPoint_Pad_D1.0mm, F.Cu at (7.53, 100.9)
- added TP606: TestPoint, TestPoint:TestPoint_Pad_D1.0mm, F.Cu at (7.53, 104.0)
- added TP607: TestPoint, TestPoint:TestPoint_Pad_D1.0mm, F.Cu at (7.53, 107.0)
- added TP608: TestPoint, Footprints:TestPoint_THTPad_D1.5mm_Drill0.7mm, F.Cu at (0.68, 108.8)
- added TP609: TestPoint, Footprints:TestPoint_THTPad_D1.5mm_Drill0.7mm, F.Cu at (0.68, 112.3)
- added TP612: TestPoint, Footprints:TestPoint_THTPad_D1.5mm_Drill0.7mm, F.Cu at (4.23, 98.1)
- added TP613: TestPoint, Footprints:TestPoint_THTPad_D1.5mm_Drill0.7mm, F.Cu at (4.23, 101.7)
- added TP616: TestPoint, Footprints:TestPoint_THTPad_D1.5mm_Drill0.7mm, F.Cu at (4.23, 105.2)
- added TP617: TestPoint, Footprints:TestPoint_THTPad_D1.5mm_Drill0.7mm, F.Cu at (4.23, 108.8)
- added TP618: TestPoint, Footprints:TestPoint_THTPad_D1.5mm_Drill0.7mm, F.Cu at (4.23, 112.3)
- added TP701: TestPoint, Footprints:TestPoint_THTPad_D1.5mm_Drill0.7mm, F.Cu at (-26.1, 98.1)
- added TP702: TestPoint, Footprints:TestPoint_THTPad_D1.5mm_Drill0.7mm, F.Cu at (-26.1, 101.7)
- added TP703: TestPoint, Footprints:TestPoint_THTPad_D1.5mm_Drill0.7mm, F.Cu at (-26.1, 105.2)
- added TP704: TestPoint, TestPoint:TestPoint_Pad_D1.0mm, F.Cu at (-19.2, 97.8)
- added TP705: TestPoint, TestPoint:TestPoint_Pad_D1.0mm, F.Cu at (-19.2, 100.9)
- added TP706: TestPoint, TestPoint:TestPoint_Pad_D1.0mm, F.Cu at (-19.2, 104.0)
- added TP707: TestPoint, TestPoint:TestPoint_Pad_D1.0mm, F.Cu at (-19.2, 107.0)
- added TP708: TestPoint, Footprints:TestPoint_THTPad_D1.5mm_Drill0.7mm, F.Cu at (-26.1, 108.8)
- added TP709: TestPoint, Footprints:TestPoint_THTPad_D1.5mm_Drill0.7mm, F.Cu at (-26.1, 112.3)
- added TP712: TestPoint, Footprints:TestPoint_THTPad_D1.5mm_Drill0.7mm, F.Cu at (-22.5, 98.1)
- added TP713: TestPoint, Footprints:TestPoint_THTPad_D1.5mm_Drill0.7mm, F.Cu at (-22.5, 101.7)
- added TP716: TestPoint, Footprints:TestPoint_THTPad_D1.5mm_Drill0.7mm, F.Cu at (-22.5, 105.2)
- added TP717: TestPoint, Footprints:TestPoint_THTPad_D1.5mm_Drill0.7mm, F.Cu at (-22.5, 108.8)
- added TP718: TestPoint, Footprints:TestPoint_THTPad_D1.5mm_Drill0.7mm, F.Cu at (-22.5, 112.3)
- added TP801: TestPoint, Footprints:TestPoint_THTPad_D1.5mm_Drill0.7mm, F.Cu at (-26.1, 124.2)
- added TP802: TestPoint, Footprints:TestPoint_THTPad_D1.5mm_Drill0.7mm, F.Cu at (-26.1, 127.8)
- added TP803: TestPoint, Footprints:TestPoint_THTPad_D1.5mm_Drill0.7mm, F.Cu at (-26.1, 131.3)
- added TP804: TestPoint, TestPoint:TestPoint_Pad_D1.0mm, F.Cu at (-19.2, 124.0)
- added TP805: TestPoint, TestPoint:TestPoint_Pad_D1.0mm, F.Cu at (-19.2, 127.0)
- added TP806: TestPoint, TestPoint:TestPoint_Pad_D1.0mm, F.Cu at (-19.2, 130.1)
- added TP807: TestPoint, TestPoint:TestPoint_Pad_D1.0mm, F.Cu at (-19.2, 133.1)
- added TP808: TestPoint, Footprints:TestPoint_THTPad_D1.5mm_Drill0.7mm, F.Cu at (-26.1, 134.8)
- added TP809: TestPoint, Footprints:TestPoint_THTPad_D1.5mm_Drill0.7mm, F.Cu at (-26.1, 138.4)
- added TP812: TestPoint, Footprints:TestPoint_THTPad_D1.5mm_Drill0.7mm, F.Cu at (-22.5, 124.2)
- added TP813: TestPoint, Footprints:TestPoint_THTPad_D1.5mm_Drill0.7mm, F.Cu at (-22.5, 127.8)
- added TP816: TestPoint, Footprints:TestPoint_THTPad_D1.5mm_Drill0.7mm, F.Cu at (-22.5, 131.3)
- added TP817: TestPoint, Footprints:TestPoint_THTPad_D1.5mm_Drill0.7mm, F.Cu at (-22.5, 134.8)
- added TP818: TestPoint, Footprints:TestPoint_THTPad_D1.5mm_Drill0.7mm, F.Cu at (-22.5, 138.4)
- added TP901: TestPoint, Footprints:TestPoint_THTPad_D1.5mm_Drill0.7mm, F.Cu at (-13.9, 124.2)
- added TP902: TestPoint, Footprints:TestPoint_THTPad_D1.5mm_Drill0.7mm, F.Cu at (-13.9, 127.8)
- added TP903: TestPoint, Footprints:TestPoint_THTPad_D1.5mm_Drill0.7mm, F.Cu at (-13.9, 131.3)
- added TP904: TestPoint, Footprints:TestPoint_THTPad_D1.5mm_Drill0.7mm, F.Cu at (-13.9, 134.8)
- moved TP410 172.5 mm to (-8.35, 127.8), turned to 0 degrees
- moved TP409 169.3 mm to (-8.35, 124.2), turned to 0 degrees
- moved JP402 40.3 mm to (108.5, 70.3), turned to -90 degrees
- moved F201 21.8 mm to (71.0, 174.0)
- moved J101 8.38 mm to (49.0, 169.2)
- moved JP417 0.80 mm to (135.2, 39.0)
- moved TP403 0.30 mm to (108.8, 56.5)
- moved TP404 0.30 mm to (108.8, 51.4)
- moved TP407 0.30 mm to (108.8, 59.0)
- moved TP408 0.30 mm to (108.8, 53.9)
Connections:
- H104 pad 1: (no net) -> Earth_Protective (x5)
- J101 pad 1: /High_side/V_{IHighIN} -> PGND
- J101 pad 2: /High_side/V_{IHighIN} -> PGND
- J101 pad 3: PGND -> /High_side/V_{IHighIN}
- J101 pad 4: PGND -> /High_side/V_{IHighIN}
- U901 pad 12: /HALL1 -> /HALL3
Routing:
- net /I_{I1Low_sense}: track 115.4 -> 21.5 mm, vias 2 -> 1
- net /Feeder/VIN: track 0.00 -> 55.3 mm, vias 252 -> 268
- net (no net): track 250.3 -> 201.6 mm, vias 6 -> 2
- net +5V_DGND: track 56.0 -> 97.4 mm, vias 20 -> 22
- net /I_{I2Low_sense}: track 52.0 -> 17.9 mm, vias 1 -> 0
- net Net-(JP417-B): track 50.2 -> 16.5 mm
- net /HRTIM_CHE2: track 172.3 -> 142.4 mm
- net Net-(D401-K): track 52.7 -> 25.4 mm
- net /MCU/PWR_COM1: track 0.00 -> 24.6 mm
- net Net-(U606--): track 0.00 -> 12.4 mm
- net DGND: track 75.1 -> 87.0 mm, vias 88 -> 78
- net /V_{I1Low_sense}: track 182.6 -> 172.0 mm, vias 3 -> 1
- net Net-(U204--): track 1.74 -> 9.54 mm, vias 0 -> 2
- net /V_{I2Low_sense}: track 56.5 -> 50.2 mm, vias 2 -> 1
- net Net-(U203--): track 0.00 -> 6.22 mm
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
Commit message: Heavy changes on the schematic and on the preliminary routing files
Signed-off-by: Jean Alinei <jean.alinei@laas.fr>
Parts:
- removed C205, C206, C208, C210, C211, C212: 33uF, Capacitor_SMD:CP_Elec_10x10.5
- removed C301, C302, C303, C304, C305: 10uF, Footprints:C_1210_3225Metric
- removed C306, C307: 1uF, Footprints:C_0805_2012Metric
- removed C414, C416: 20pF, Footprints:C_0805_2012Metric
- removed C415: 100nF, Footprints:C_0805_2012Metric
- removed D401, D402: RBR2MM60ATFTR, Diode_SMD:D_SOD-123
- removed J405, J406: Conn_01x02_Male, Connector_JST:JST_EH_B2B-EH-A_1x02_P2.50mm_Vertical
- removed JP407: SolderJumper_2_Open, Jumper:SolderJumper-2_P1.3mm_Bridged_Pad1.0x1.5mm
- removed JP411: Jumper_2_Bridged, Jumper:SolderJumper-2_P1.3mm_Open_Pad1.0x1.5mm
- removed L301: 22uH, Inductor_SMD:L_1210_3225Metric
- removed L601, L701, L801: 8,2uH, Footprints:SRP1510CA-330M
- removed N101: Housing_Pad, Footprints:Guard_ring
- removed PS301: TBA 1-0512, Footprints:Converter_DCDC_Murata_MEE1SxxxxSC_THT
- removed R301: 1R, Footprints:R_0805_2012Metric
- removed R422: 47k, Footprints:R_0805_2012Metric
- removed R423: 12k, Footprints:R_0805_2012Metric
- removed U301: AP1117-50, Package_TO_SOT_SMD:SOT-223-3_TabPin2
- removed U302: MCP1799T-5002H/TT, Footprints:SOT-23_copy
- removed U407: OPA316, Package_TO_SOT_SMD:SOT-353_SC-70-5
- added C522: 10uF, Footprints:C_1210_3225Metric, F.Cu at (82.4, 44.0)
- added C523: 10uF, Footprints:C_1210_3225Metric, F.Cu at (94.0, 54.6)
- added C524: 10uF, Footprints:C_1210_3225Metric, F.Cu at (203.0, 97.6)
- added C525: 10uF, Footprints:C_1210_3225Metric, F.Cu at (206.0, 97.6)
- added C526: 10uF, Footprints:C_1210_3225Metric, F.Cu at (206.0, 106.4)
- added C527: 1uF, Footprints:C_0805_2012Metric, F.Cu at (210.7, 111.3)
- added C528: 1uF, Footprints:C_0805_2012Metric, F.Cu at (210.7, 116.3)
- added C529: 20pF, Footprints:C_0805_2012Metric, F.Cu at (187.9, 75.1)
- added C530: 100nF, Footprints:C_0805_2012Metric, F.Cu at (193.9, 77.1)
- added C531: 20pF, Footprints:C_0805_2012Metric, F.Cu at (190.9, 80.0)
- added J401: Conn_01x02_Male, Connector_JST:JST_EH_B2B-EH-A_1x02_P2.50mm_Vertical, F.Cu at (53.0, 25.0)
- added J402: Conn_01x02_Male, Connector_JST:JST_EH_B2B-EH-A_1x02_P2.50mm_Vertical, F.Cu at (57.0, 27.5)
- added JP502: SolderJumper_2_Open, Jumper:SolderJumper-2_P1.3mm_Bridged_Pad1.0x1.5mm, F.Cu at (194.3, 80.1)
- added L503: 22uH, Inductor_SMD:L_1210_3225Metric, F.Cu at (204.6, 101.6)
- added PS501: TBA 1-0512, Footprints:Converter_DCDC_Murata_MEE1SxxxxSC_THT, F.Cu at (210.0, 99.0)
- added R519: 1R, Footprints:R_0805_2012Metric, F.Cu at (94.0, 51.1)
- added R520: 47k, Footprints:R_0805_2012Metric, F.Cu at (191.0, 74.1)
- added R521: 12k, Footprints:R_0805_2012Metric, F.Cu at (185.9, 75.0)
- added U504: AP1117-50, Package_TO_SOT_SMD:SOT-223-3_TabPin2, F.Cu at (89.0, 51.0)
- added U505: MCP1799T-5002H/TT, Footprints:SOT-23_copy, F.Cu at (210.9, 114.0)
- added U506: OPA316, Package_TO_SOT_SMD:SOT-353_SC-70-5, F.Cu at (190.9, 77.1)
- moved H102 209.3 mm to (202.0, 152.8)
- moved H109 209.3 mm to (202.0, 159.0)
- moved H104 129.7 mm to (185.0, 170.0)
- moved H104 129.7 mm to (212.8, 170.0)
- moved H104 129.7 mm to (240.9, 169.8)
- moved C720 88.9 mm to (52.0, 120.4), turned to 180 degrees
- moved C721 88.9 mm to (52.0, 132.4), turned to 180 degrees
- moved C820 88.6 mm to (52.0, 145.1), turned to 180 degrees
- moved C821 88.6 mm to (52.0, 157.1), turned to 180 degrees
- moved C620 60.6 mm to (52.0, 96.0), turned to 180 degrees
- moved C621 60.6 mm to (52.0, 108.0), turned to 180 degrees
- moved JP406 26.8 mm to (135.3, 31.0), turned to 0 degrees
- moved D605 16.2 mm to (79.0, 108.0), turned to 180 degrees
- moved D805 16.1 mm to (134.0, 108.0), turned to 180 degrees
- moved D705 16.1 mm to (106.0, 108.0), turned to 180 degrees
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Connections:
- C411 pad 1: /MCU/ADC2_IN5 -> Net-(C411-Pad1)
- C608 pad 1: /Feeder/VIN -> /High_side/V_{IHigh}
- C609 pad 1: /Feeder/VIN -> /High_side/V_{IHigh}
- C620 pad 1: /Feeder/VIN -> /High_side/V_{IHigh}
- C621 pad 1: /Feeder/VIN -> /High_side/V_{IHigh}
- C622 pad 1: /Feeder/VIN -> /High_side/V_{IHigh}
- C624 pad 1: /Feeder/VIN -> /High_side/V_{IHigh}
- C626 pad 1: /Feeder/VIN -> /High_side/V_{IHigh}
- C708 pad 1: /Feeder/VIN -> /High_side/V_{IHigh}
- C709 pad 1: /Feeder/VIN -> /High_side/V_{IHigh}
- C720 pad 1: /Feeder/VIN -> /High_side/V_{IHigh}
- C721 pad 1: /Feeder/VIN -> /High_side/V_{IHigh}
- C722 pad 1: /Feeder/VIN -> /High_side/V_{IHigh}
- C724 pad 1: /Feeder/VIN -> /High_side/V_{IHigh}
- C726 pad 1: /Feeder/VIN -> /High_side/V_{IHigh}
- C808 pad 1: /Feeder/VIN -> /High_side/V_{IHigh}
- C809 pad 1: /Feeder/VIN -> /High_side/V_{IHigh}
- C820 pad 1: /Feeder/VIN -> /High_side/V_{IHigh}
- C821 pad 1: /Feeder/VIN -> /High_side/V_{IHigh}
- C822 pad 1: /Feeder/VIN -> /High_side/V_{IHigh}
- C824 pad 1: /Feeder/VIN -> /High_side/V_{IHigh}
- C826 pad 1: /Feeder/VIN -> /High_side/V_{IHigh}
- F201 pad 1: /High_side/V_{IHighIN} -> /Feeder/VIN
- F401 pad 1: /MCU/PWR_COM1 -> /Feeder/PWR_COM1
- F401 pad 2: Net-(D401-K) -> +6V
- F402 pad 1: /MCU/PWR_COM2 -> /Feeder/PWR_COM2
- F402 pad 2: Net-(D401-K) -> +6V
- H104 pad 1: (no net) -> Earth_Protective (x2)
- J101 pad 3: /High_side/V_{IHighIN} -> /Feeder/VIN
- J101 pad 4: /High_side/V_{IHighIN} -> /Feeder/VIN
- JP404 pad 1: /MCU/PC13 -> /High_side/V_{IHigh}
- JP405 pad 1: /MCU/PC6 -> /High_side/V_{IHigh}
- JP417 pad 1: /MCU/DAC2 -> /High_side/V_{IHigh}
- Q601 pad 2: /Feeder/VIN -> /High_side/V_{IHigh}
- Q602 pad 1: Net-(D601-A) -> /High_side/V_{IHigh}
- Q701 pad 2: /Feeder/VIN -> /High_side/V_{IHigh}
- Q801 pad 2: /Feeder/VIN -> /High_side/V_{IHigh}
- R201 pad 1: /Feeder/VIN -> /High_side/V_{IHigh}
- R407 pad 1: /MCU/Temp2 -> /High_side/V_{IHigh}
- R415 pad 1: /MCU/ADC2_IN5 -> Net-(C411-Pad1)
- R470 pad 2: Net-(R470-Pad2) -> Net-(C411-Pad1)
- R608 pad 2: Net-(D601-A) -> /High_side/V_{IHigh}
- R622 pad 1: /Feeder/VIN -> /High_side/V_{IHigh}
- R722 pad 1: /Feeder/VIN -> /High_side/V_{IHigh}
- R822 pad 1: /Feeder/VIN -> /High_side/V_{IHigh}
- TH402 pad 1: /MCU/Temp2 -> /High_side/V_{IHigh}
- TH403 pad 1: /MCU/Temp3 -> /High_side/V_{IHigh}
- U202 pad 1: /Feeder/VIN -> /High_side/V_{IHigh}
- U202 pad 2: /Feeder/VIN -> /High_side/V_{IHigh}
- U401 pad 14: /HRTIM_CHA1 -> /High_side/V_{IHigh}
- U401 pad 15: /MCU/Temp3_Mux -> /High_side/V_{IHigh}
- U401 pad 16: /MCU/USART3_TX -> /High_side/V_{IHigh}
- U401 pad 17: /MCU/USART3_RX -> /High_side/V_{IHigh}
- U401 pad 18: DGND -> /High_side/V_{IHigh}
- U401 pad 19: /MCU/PC12 -> /High_side/V_{IHigh}
- U401 pad 20: /MCU/CAN1_STB -> /High_side/V_{IHigh}
- U401 pad 26: /V_{IHigh_sense} -> /High_side/V_{IHigh}
- U401 pad 27: /I_{IHigh_sense} -> /High_side/V_{IHigh}
- U401 pad 28: DGND -> /High_side/V_{IHigh}
- U401 pad 29: /V_{I2Low_sense} -> /High_side/V_{IHigh}
- U401 pad 30: /I_{I2Low_sense} -> /High_side/V_{IHigh}
- U401 pad 31: /MCU/Neutral_buff -> /High_side/V_{IHigh}
- U401 pad 32: unconnected-(U401A-PA5-Pad32) -> /High_side/V_{IHigh}
- U401 pad 33: DGND -> /High_side/V_{IHigh}
- U401 pad 34: /MCU/DAC2 -> /High_side/V_{IHigh}
- U401 pad 35: /MCU/ADC2_IN5 -> /High_side/V_{IHigh}
- U401 pad 36: +3.3V_DGND -> /High_side/V_{IHigh}
- U401 pad 50: unconnected-(U401C-PB3-Pad50) -> /High_side/V_{IHigh}
- U401 pad 51: unconnected-(U401C-PA2-Pad51) -> /High_side/V_{IHigh}
- U401 pad 59: unconnected-(U401D-RST-Pad59) -> /High_side/V_{IHigh}
- U402 pad 1: /MCU/FDCAN1_{TX} -> /High_side/V_{IHigh}
- U402 pad 4: /MCU/FDCAN1_{RX} -> /High_side/V_{IHigh}
- U405 pad 1: /MCU/USART3_RX -> /High_side/V_{IHigh}
- U405 pad 4: /MCU/USART3_TX -> /High_side/V_{IHigh}
- U406 pad 7: Net-(R470-Pad2) -> Net-(C411-Pad1)
- U605 pad 1: Net-(L601-Pad1) -> /Phase1/SW_Node
- U605 pad 2: Net-(L601-Pad1) -> /Phase1/SW_Node
- U705 pad 1: Net-(L701-Pad1) -> /Phase2/SW_Node
- U705 pad 2: Net-(L701-Pad1) -> /Phase2/SW_Node
- U805 pad 1: Net-(L801-Pad1) -> /Phase3/SW_Node
- U805 pad 2: Net-(L801-Pad1) -> /Phase3/SW_Node
Routing:
- net /MCU/PC13: track 205.4 -> 0.00 mm, vias 1 -> 0
- net /Phase1/SW_Node: track 203.2 -> 0.00 mm, vias 48 -> 45
- net (no net): track 201.6 -> 2.66 mm, vias 2 -> 0
- net /V_{I1Low_sense}: track 172.0 -> 7.01 mm
- net /HRTIM_CHA1: track 187.6 -> 25.7 mm, vias 1 -> 0
- net /HRTIM_CHA2: track 182.6 -> 30.4 mm
- net /HRTIM_CHE2: track 142.4 -> 0.00 mm
- net /HRTIM_CHE1: track 141.8 -> 0.00 mm
- net Net-(F801-Pad1): track 143.8 -> 3.15 mm
- net /I_{IHigh_sense}: track 145.5 -> 7.53 mm
- net /HRTIM_CHC2: track 172.3 -> 51.0 mm
- net /~{STBY1}: track 101.4 -> 0.00 mm, vias 6 -> 0
- net /MCU/Temp3: track 97.6 -> 1.03 mm, vias 2 -> 1
- net Net-(F701-Pad1): track 91.4 -> 0.00 mm
- net /High_side/V_{IHigh}: track 0.00 -> 85.3 mm, vias 0 -> 291
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- added copper zone on F.Cu, net +5V_DGND
- added copper zone on B.Cu, net /High_side/V_{IHigh}
- added copper zone on F.Cu, net /High_side/V_{IHigh}
- added copper zone on In3.Cu, net /High_side/V_{IHigh}
- added copper zone on In4.Cu, net DGND
- added copper zone on F.Cu, net Net-(D507-A)
- removed copper zone on F.Cu, net (none)
- removed copper zone on B.Cu, net /Feeder/VIN
- removed copper zone on F.Cu, net /High_side/V_{IHighIN}
- removed copper zone on In3.Cu, net /High_side/V_{IHighIN}
- removed copper zone on F.Cu, net /Phase1/SW_Node
- removed copper zone on F.Cu, net /Phase2/SW_Node
- removed copper zone on F.Cu, net /Phase3/SW_Node
- removed copper zone on F.Cu, net Net-(L601-Pad1)
- removed copper zone on F.Cu, net Net-(L701-Pad1)
- removed copper zone on F.Cu, net Net-(L801-Pad1)
