File: KiCAD_files/inverter.kicad_pcb (KiCad board)
At the start: 6 copper layers, 100 x 160 mm, 463 parts, among them J101 Wago 4 contacts, J103 Wago 6 contacts, J104 2604-1102, J106 2604-1102, J108 2604-1102, J401 Conn_01x02_Male, J402 Conn_01x02_Male, J403 RJ45_LED_Shielded, J404 RJ45_LED_Shielded, J501 Conn_01x03, J901 Conn_01x05, Q501 60V N channel, Q502 TK13P25D,RQ, Q601 IPD200N15N3, Q602 IPD200N15N3, Q701 IPD200N15N3, Q702 IPD200N15N3, Q801 IPD200N15N3, Q802 IPD200N15N3, T501 PA2467NL, U201 AMC1311DWV, U202 +-20A Hall, U203 OPA316, U204 OPA316, U401 OwnTech_SPIN, U402 TCAN334GDR, U405 LTC2850xS8, U406 OPA2277, U410 TS5A3357DCUT, U490 OPA316, U501 NCP12700, U502 FODM217A, U503 TL431MFDT,215, U504 AP1117-50, U505 MCP1799T-5002H/TT, U506 OPA316, U601 AMC1100DUB, U602 FODM217A, U603 UCC21222DR, U604 OPA316, U605 ACS730KLCTR-20AB, U606 OPA316, U701 AMC1100DUB, U702 FODM217A, U703 UCC21222DR, U704 OPA316, U705 ACS730KLCTR-20AB, U706 OPA316, U801 AMC1100DUB, U802 FODM217A, U803 UCC21222DR, U804 OPA316, U805 ACS730KLCTR-20AB, U806 OPA316, U901 Si8640BB-B-IS1

Commit message: Added the Harting footprint with WAGO support. Improved component placement.
Signed-off-by: Jean Alinei <jean.alinei@laas.fr>
Parts:
- removed the H104 at (136.4, 156.0)
- removed the H104 at (240.9, 169.8)
- removed J103: Wago 6 contacts, Footprints:WAGO-2604-1106
- removed J104, J106, J108: 2604-1102, Footprints:WAGO-2604-1102
- added N101: Housing_Pad, Footprints:Guard_ring, F.Cu at (42.0, 22.0)
- J101: value Wago 4 contacts -> Harting-15 and Wago 6; footprint Footprints:WAGO-2604-1104 -> Footprints:Harting - 15contacts and Wago
- moved H102 314.7 mm to (-29.0, -61.0)
- moved H109 314.7 mm to (-29.0, -54.8)
- moved C528 144.3 mm to (71.0, 80.1), turned to -90 degrees
- moved U505 141.6 mm to (73.4, 80.3), turned to -90 degrees
- moved C527 138.3 mm to (76.0, 80.1), turned to 90 degrees
- moved C526 128.8 mm to (80.6, 77.0), turned to 0 degrees
- moved PS501 123.3 mm to (88.0, 81.0), turned to -90 degrees
- moved L503 122.0 mm to (85.4, 75.6), turned to -90 degrees
- moved C525 118.4 mm to (89.4, 77.0), turned to 0 degrees
- moved C524 116.0 mm to (89.4, 74.0), turned to 0 degrees
- moved H104 85.9 mm to (137.5, 128.5)
- moved H104 83.5 mm to (112.5, 128.5)
- moved JP502 82.0 mm to (112.3, 77.0), turned to 180 degrees
- moved C530 81.3 mm to (112.7, 80.0), turned to 90 degrees
- moved R426 79.2 mm to (136.0, 82.0)
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Connections:
- C608 pad 1: /High_side/V_{IHigh} -> /Feeder/VIN
- C609 pad 1: /High_side/V_{IHigh} -> /Feeder/VIN
- C620 pad 1: /High_side/V_{IHigh} -> /Feeder/VIN
- C621 pad 1: /High_side/V_{IHigh} -> /Feeder/VIN
- C622 pad 1: /High_side/V_{IHigh} -> /Feeder/VIN
- C624 pad 1: /High_side/V_{IHigh} -> /Feeder/VIN
- C626 pad 1: /High_side/V_{IHigh} -> /Feeder/VIN
- C708 pad 1: /High_side/V_{IHigh} -> /Feeder/VIN
- C709 pad 1: /High_side/V_{IHigh} -> /Feeder/VIN
- C720 pad 1: /High_side/V_{IHigh} -> /Feeder/VIN
- C721 pad 1: /High_side/V_{IHigh} -> /Feeder/VIN
- C722 pad 1: /High_side/V_{IHigh} -> /Feeder/VIN
- C724 pad 1: /High_side/V_{IHigh} -> /Feeder/VIN
- C726 pad 1: /High_side/V_{IHigh} -> /Feeder/VIN
- C808 pad 1: /High_side/V_{IHigh} -> /Feeder/VIN
- C809 pad 1: /High_side/V_{IHigh} -> /Feeder/VIN
- C820 pad 1: /High_side/V_{IHigh} -> /Feeder/VIN
- C821 pad 1: /High_side/V_{IHigh} -> /Feeder/VIN
- C822 pad 1: /High_side/V_{IHigh} -> /Feeder/VIN
- C824 pad 1: /High_side/V_{IHigh} -> /Feeder/VIN
- C826 pad 1: /High_side/V_{IHigh} -> /Feeder/VIN
- F201 pad 1: /Feeder/VIN -> /High_side/V_{IHighIN}
- J101 pad 1: PGND -> /High_side/V_{IHighIN}
- J101 pad 2: PGND -> /High_side/V_{IHighIN}
- J101 pad 3: /Feeder/VIN -> PGND
- J101 pad 4: /Feeder/VIN -> PGND
- JP404 pad 1: /High_side/V_{IHigh} -> /MCU/PC13
- JP405 pad 1: /High_side/V_{IHigh} -> /MCU/PC6
- JP417 pad 1: /High_side/V_{IHigh} -> /MCU/DAC2
- Q601 pad 2: /High_side/V_{IHigh} -> /Feeder/VIN
- Q602 pad 1: /High_side/V_{IHigh} -> Net-(D601-A)
- Q701 pad 2: /High_side/V_{IHigh} -> /Feeder/VIN
- Q801 pad 2: /High_side/V_{IHigh} -> /Feeder/VIN
- R201 pad 1: /High_side/V_{IHigh} -> /Feeder/VIN
- R407 pad 1: /High_side/V_{IHigh} -> /MCU/Temp2
- R608 pad 2: /High_side/V_{IHigh} -> Net-(D601-A)
- R622 pad 1: /High_side/V_{IHigh} -> /Feeder/VIN
- R722 pad 1: /High_side/V_{IHigh} -> /Feeder/VIN
- R822 pad 1: /High_side/V_{IHigh} -> /Feeder/VIN
- TH402 pad 1: /High_side/V_{IHigh} -> /MCU/Temp2
- TH403 pad 1: /High_side/V_{IHigh} -> /MCU/Temp3
- U202 pad 1: /High_side/V_{IHigh} -> /Feeder/VIN
- U202 pad 2: /High_side/V_{IHigh} -> /Feeder/VIN
- U401 pad 14: /High_side/V_{IHigh} -> /HRTIM_CHA1
- U401 pad 15: /High_side/V_{IHigh} -> /MCU/Temp3_Mux
- U401 pad 16: /High_side/V_{IHigh} -> /MCU/USART3_TX
- U401 pad 17: /High_side/V_{IHigh} -> /MCU/USART3_RX
- U401 pad 18: /High_side/V_{IHigh} -> DGND
- U401 pad 19: /High_side/V_{IHigh} -> /MCU/PC12
- U401 pad 20: /High_side/V_{IHigh} -> /MCU/CAN1_STB
- U401 pad 26: /High_side/V_{IHigh} -> /V_{IHigh_sense}
- U401 pad 27: /High_side/V_{IHigh} -> /I_{IHigh_sense}
- U401 pad 28: /High_side/V_{IHigh} -> DGND
- U401 pad 29: /High_side/V_{IHigh} -> /V_{I2Low_sense}
- U401 pad 30: /High_side/V_{IHigh} -> /I_{I2Low_sense}
- U401 pad 31: /High_side/V_{IHigh} -> /MCU/Neutral_buff
- U401 pad 32: /High_side/V_{IHigh} -> unconnected-(U401A-PA5-Pad32)
- U401 pad 33: /High_side/V_{IHigh} -> DGND
- U401 pad 34: /High_side/V_{IHigh} -> /MCU/DAC2
- U401 pad 35: /High_side/V_{IHigh} -> /MCU/ADC2_IN5
- U401 pad 36: /High_side/V_{IHigh} -> +3.3V_DGND
- U401 pad 50: /High_side/V_{IHigh} -> unconnected-(U401C-PB3-Pad50)
- U401 pad 51: /High_side/V_{IHigh} -> unconnected-(U401C-PA2-Pad51)
- U401 pad 59: /High_side/V_{IHigh} -> unconnected-(U401D-RST-Pad59)
- U402 pad 1: /High_side/V_{IHigh} -> /MCU/FDCAN1_{TX}
- U402 pad 4: /High_side/V_{IHigh} -> /MCU/FDCAN1_{RX}
- U405 pad 1: /High_side/V_{IHigh} -> /MCU/USART3_RX
- U405 pad 4: /High_side/V_{IHigh} -> /MCU/USART3_TX
Routing:
- net /High_side/V_{IHigh}: track 85.3 -> 0.00 mm, vias 291 -> 0
- net /MCU/PWR_COM2: track 47.0 -> 0.00 mm, vias 1 -> 0
- net +3.3V_DGND: track 44.6 -> 6.37 mm
- net /MCU/PWR_COM1: track 24.6 -> 0.00 mm
- net /Hall_Sensor/HALL3_PGND: track 26.0 -> 1.62 mm
- net (no net): track 2.66 -> 24.5 mm
- net /Hall_Sensor/HALL2_PGND: track 20.1 -> 1.39 mm
- net /MCU/USART3_RX: track 0.00 -> 17.8 mm
- net +6V: track 20.1 -> 2.66 mm, vias 7 -> 6
- net /MCU/USART3_TX: track 0.00 -> 17.4 mm, vias 0 -> 200
- net /Hall_Sensor/HALL1_PGND: track 15.0 -> 1.39 mm
- net DGND: track 65.7 -> 54.0 mm, vias 45 -> 29
- net +5V_DGND: track 52.4 -> 45.9 mm, vias 16 -> 6
- net Net-(U501-UVLO): track 3.52 -> 9.59 mm
- net /Feeder/input: track 23.1 -> 29.0 mm
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- added copper zone on B.Cu, net /MCU/USART3_TX
- added copper zone on F.Cu, net /Phase1/SW_Node
- added copper zone on F.Cu, net /Phase2/SW_Node
- added copper zone on F.Cu, net /Phase3/SW_Node
- added copper zone on In1.Cu, net DGND
- added copper zone on In2.Cu, net Net-(F601-Pad1)
- added copper zone on In2.Cu, net Net-(F701-Pad1)
- added copper zone on In2.Cu, net Net-(F801-Pad1)
- added copper zone on In1.Cu, net PGND
- removed copper zone on B.Cu, net +12V_PGND
- removed copper zone on B.Cu, net /High_side/V_{IHigh}
- removed copper zone on F.Cu, net /High_side/V_{IHigh}
- removed copper zone on In3.Cu, net /High_side/V_{IHigh}
- removed copper zone on In3.Cu, net /MCU/GND_COM
- removed copper zone on F.Cu, net /Phase A
- removed copper zone on In3.Cu, net /Phase A
- removed copper zone on F.Cu, net /Phase B
- removed copper zone on In3.Cu, net /Phase B
- removed copper zone on F.Cu, net /Phase C
- removed copper zone on In3.Cu, net /Phase C
Other:
- board text removed: "-"
- board text removed: "11-120V_{IN} 6V_{OUT} @ 0.5A"
- board text removed: "DGND"
